File: pcb/tropic01-universal-secure-device/kicad/tropic01-universal-secure-device.kicad_pcb (KiCad board)
At the start: 6 copper layers, 42.7 x 36 mm, 90 parts, among them J1 USB4105-GF-A, J2 ER-TFT024IPS-3 50P FFC, J6 SM04B-SRSS-TB, J9 S2B-PH-SM4-TB, SW1 EVQP7J01P, U1 STM32U585VIT6, U10 BQ24074RGTR, U11 OPTIGA-TRUST-M-SLS32AIA, U13 TPS22917DBVR, U14 TPS22917DBVR, U15 TPS61165DBVR, U2 TR01-C2P-T301, U3 TPS62840DLCR, U4 TPS22917DBVR, U5 W25Q128JVSIQ, U7 TPD4E05U06DQAR, U8 TPS2553DBVR, U9 ST25R3916B-AQET, X1 16MHz, X3 FA-238 27.12MHz

Commit message: refactor(pcb): improve floorplan - TROPIC01 by STM32, J2 to center
Review-driven placement fixes on the 42.87x36 floorplan:
- TROPIC01 (U2, secure element) moved adjacent to the STM32 (U1) - the secure
  SPI bus was crossing the whole board (U2 was on the far-left edge, ~12mm away);
  now edge-to-edge (~1mm gap) for a short bus.
- J2 (display FFC) moved from the bottom edge to the board CENTER: the display's
  FPC tail exits the display bottom and folds UNDER the screen, so the connector
  end lands ~25mm up (per datasheet) = mid-board, not at the bottom.
- NFC IC (U9) nudged off the battery connector J9 (resolved the last overlap).
- 0 courtyard/clearance overlaps; 78/78 placed; all perimeter + two-sided
  constraints still respected (display side = only J2).

Remaining DRC = cosmetic silk + inherent edge-mounted-connector clearance,
addressed in the pre-gerber pass.
Parts:
- moved C6 35.3 mm to (43.7, 61.4)
- moved C8 32.1 mm to (27.7, 35.0)
- moved R5 32.0 mm to (41.7, 63.0)
- moved C3 31.6 mm to (41.3, 59.8)
- moved C4 30.6 mm to (41.3, 61.4)
- moved TP_GND 30.6 mm to (45.8, 61.6)
- moved C5 30.1 mm to (41.3, 58.2)
- moved TP_3V3 29.9 mm to (43.8, 63.2)
- moved C17 28.1 mm to (41.7, 64.6)
- moved U4 25.8 mm to (37.7, 59.5)
- moved U2 25.2 mm to (39.0, 54.5)
- moved TP_UART_TX 24.1 mm to (15.8, 59.6)
- moved R9 22.0 mm to (48.5, 56.6)
- moved U13 21.9 mm to (33.7, 37.9)
- moved C7 21.6 mm to (13.7, 46.2)
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