File: pcb/tropic01-universal-secure-device/kicad/tropic01-universal-secure-device.kicad_pcb (KiCad board)
At the start: 4 copper layers, 42.7 x 36 mm, 90 parts, among them J1 USB4105-GF-A, J2 ER-TFT024IPS-3 50P FFC, J6 SM04B-SRSS-TB, J7 SWD_TC2030, J9 S2B-PH-SM4-TB, SW1 EVQP7J01P, U1 STM32U585VIT6, U10 BQ24074RGTR, U11 OPTIGA-TRUST-M-SLS32AIA, U13 TPS22917DBVR, U14 TPS22917DBVR, U15 TPS61165DBVR, U2 TR01-C2P-T301, U3 TPS62840DLCR, U4 TPS22917DBVR, U5 W25Q128JVSIQ, U7 TPD4E05U06DQAR, U8 TPS2553DBVR, U9 ST25R3916B-AQET, X1 16MHz, X3 FA-238 27.12MHz

Commit message: feat(pcb): BOOT0 jumper + grouped UART + per-rail current-sense jumpers
- BOOT0: JP1 solder-jumper (BOOT0<->SYS_3V3), normally open; set + power-cycle for
  USB-DFU. R22 100k keeps BOOT0 low normally. No BOOT0 button.
- UART console grouped: TP_UART_TX/RX relocated next to a new TP_UART_GND.
- Current-sense: split TROPIC_VCC_SW (RJ1) and NFC_VCC_SW (RJ2) with series 0R
  jumpers so each secure element's supply current is measurable.
- Holistic re-placement to fit the new parts (board at capacity); GND plane
  refilled. DRC hard violations = only the 2 accepted USB-C edge posts; back side
  still carries only J2.

Power-latch (SW1 true-off) intentionally NOT auto-wired: it needs power-tree
surgery + the TPS62840 EN pinout, a critical path to be designed/validated in the
schematic (see spec). Board keeps safe always-on power for now.
Parts:
- added JP1: BOOT0_DFU, SolderJumper-2_P1.3mm_Open_Pad1.0x1.5mm, F.Cu at (24.3, 67.2)
- added RJ1: 0R, R_0402_1005Metric, F.Cu at (36.0, 59.9)
- added RJ2: 0R, R_0402_1005Metric, F.Cu at (38.5, 59.9)
- added TP_UART_GND: GND, TestPoint_Pad_D1.0mm, F.Cu at (36.1, 58.0)
- moved C19 24.4 mm to (36.0, 53.0)
- moved TP_UART_RX 22.9 mm to (35.7, 54.6)
- moved TP_UART_TX 21.3 mm to (35.7, 56.1)
- moved C18 9.01 mm to (12.5, 60.5)
- moved L15 5.83 mm to (49.0, 58.0)
- moved TP_BOOT0 5.15 mm to (17.0, 62.0)
- moved C41 4.27 mm to (44.5, 56.0)
- moved C16 3.64 mm to (14.0, 65.5)
- moved C17 3.50 mm to (16.5, 68.0)
- moved R5 3.50 mm to (16.5, 66.5)
- moved X1 3.50 mm to (20.0, 67.5)
- moved R12 1.00 mm to (52.0, 58.5)
- moved R14 1.00 mm to (52.0, 57.0)
- moved R16 1.00 mm to (48.5, 60.0)
- moved U2 1.00 mm to (40.0, 55.0)
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Connections:
- C3 pad 1: TROPIC_VCC_SW -> TROPIC_VCC
- C4 pad 1: TROPIC_VCC_SW -> TROPIC_VCC
- C41 pad 1: NFC_VCC_SW -> NFC_VCC
- C5 pad 1: TROPIC_VCC_SW -> TROPIC_VCC
- U2 pad 1: TROPIC_VCC_SW -> TROPIC_VCC
- U2 pad 11: TROPIC_VCC_SW -> TROPIC_VCC
- U2 pad 22: TROPIC_VCC_SW -> TROPIC_VCC
- U2 pad 24: TROPIC_VCC_SW -> TROPIC_VCC
- U9 pad 1: NFC_VCC_SW -> NFC_VCC
- U9 pad 10: NFC_VCC_SW -> NFC_VCC
- U9 pad 14: NFC_VCC_SW -> NFC_VCC
- U9 pad 8: NFC_VCC_SW -> NFC_VCC
