File: pcb/tropic01-universal-secure-device/kicad/tropic01-universal-secure-device.kicad_pcb (KiCad board)
At the start: 4 copper layers, 42.7 x 39.8 mm, 102 parts, among them J1 USB4105-GF-A, J2 ER-TFT024IPS-3 50P FFC, J6 SM04B-SRSS-TB, J7 SWD_TC2030, J9 S2B-PH-SM4-TB, SW1 EVQP7J01P, U1 STM32U585VIT6, U10 BQ24074RGTR, U11 OPTIGA-TRUST-M-SLS32AIA, U13 TPS22917DBVR, U14 TPS22917DBVR, U15 TPS61165DBVR, U2 TR01-C2P-T301, U3 TPS62840DLCR, U4 TPS22917DBVR, U5 W25Q128JVSIQ, U7 TPD4E05U06DQAR, U8 TPS2553DBVR, U9 ST25R3916B-AQET, X1 16MHz, X3 FA-238 27.12MHz

Commit message: fix(pcb): place VCAP cap + resolve I2C conflict + re-route (DRC 0)
Resolved both critical audit bugs:
- VCAP: added C59 (4.7uF) on a dedicated VCAP net, 1.9mm from STM32 pin48,
  via a full re-place that reserves the room (all 9 VDD decoupling 1.9-3.5mm,
  VCAP 1.9mm).
- I2C conflict: merged EXP/Qwiic (J6) onto the TOUCH I2C1 bus (multi-drop);
  OPTIGA secure element stays isolated on I2C4; PB10/PD13 freed. No conflict.
Full re-place (103 footprints) + re-route: 926 tracks + 129 vias, ~85%
(158/187), DRC = 0. Remaining 29 nets for the interactive router; power-trace
widening (net-class re-route) still pending. See design-notes/AUDIT-findings.md.
Parts:
- added C59: 4.7uF, C_0402_1005Metric, F.Cu at (32.5, 59.5)
- moved C40 23.5 mm to (38.0, 36.0)
- moved C41 12.8 mm to (50.0, 40.5)
- moved R4 7.50 mm to (37.5, 59.5)
- moved DISP1 4.00 mm to (110.0, 125.0)
- moved R3 2.50 mm to (30.0, 59.5)
- moved C14 1.50 mm to (50.0, 39.0)
- moved C34 1.50 mm to (50.0, 37.5)
Connections:
- J6 pad 3: EXP_I2C_SDA -> TOUCH_I2C_SDA
- J6 pad 4: EXP_I2C_SCL -> TOUCH_I2C_SCL
- U1 pad 47: EXP_I2C_SCL -> (no net)
- U1 pad 60: EXP_I2C_SDA -> (no net)
Routing:
- net TFT_BACKLIGHT_PWM: track 52.0 -> 0.00 mm, vias 2 -> 0
- net EXP_I2C_SCL: track 37.8 -> 0.00 mm, vias 2 -> 0
- net SYS_3V3: track 228.9 -> 258.3 mm, vias 6 -> 5
- net NRST: track 28.9 -> 0.00 mm, vias 3 -> 0
- net NFC_SPI_CSN: track 24.9 -> 0.00 mm, vias 2 -> 0
- net QSPI_IO2: track 24.7 -> 0.00 mm, vias 3 -> 0
- net NFC_VDD_AM: track 0.00 -> 24.5 mm, vias 0 -> 2
- net NFC_IRQ: track 0.00 -> 23.7 mm, vias 0 -> 2
- net VBUS_LIMITED: track 2.29 -> 25.7 mm, vias 0 -> 3
- net BTN_USER: track 60.8 -> 39.3 mm, vias 4 -> 2
- net USB_VBUS_SENSE: track 29.7 -> 49.7 mm, vias 3 -> 4
- net NFC_SPI_SCK: track 19.4 -> 0.00 mm, vias 2 -> 0
- net SE2_RST: track 32.6 -> 13.6 mm
- net QSPI_CLK: track 18.0 -> 0.00 mm, vias 2 -> 0
- net USB_DM: track 0.00 -> 17.8 mm, vias 0 -> 2
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